Commit message: Add pkgs

File: gonzo_description/urdf/gonzo.xacro (robot description, xacro)
@@ -9,139 +9,142 @@
   <inertial>
     <origin xyz="0.004369403453275925 -7.02165131943858e-05 0.06024663017842304" rpy="0 0 0"/>
-    <mass value="0.20273197769577378"/>
-    <inertia ixx="0.000438" iyy="0.000482" izz="0.000751" ixy="0.0" iyz="-0.0" ixz="7e-06"/>
-  </inertial>
-  <visual>
-    <origin xyz="0 0 0" rpy="0 0 0"/>
+    <mass value="5.20273197769577378"/>
+    <inertia ixx="0.0438" iyy="0.0482" izz="0.0751" ixy="0.0" iyz="-0.0" ixz="7e-05"/>
+  </inertial>
+  <visual>
+    <origin xyz="0 0 -0.05" rpy="0 0 0"/>
     <geometry>
       <mesh filename="package://gonzo_description/meshes/base_link.stl" scale="0.001 0.001 0.001"/>
     </geometry>
+    <material name="body_black"/>
+  </visual>
+  <collision>
+    <origin xyz="0 0 -0.05" rpy="0 0 0"/>
+    <geometry>
+      <mesh filename="package://gonzo_description/meshes/base_link.stl" scale="0.001 0.001 0.001"/>
+    </geometry>
+  </collision>
+</link>
+<link name="right_tyre">
+  <inertial>
+    <origin xyz="-9.273384193181355e-08 -0.017748789854178187 -5.2862379126827896e-08" rpy="0 0 0"/>
+    <mass value="1.109430614326367688"/>
+    <inertia ixx="5e-03" iyy="9e-03" izz="5e-03" ixy="-0.0" iyz="-0.0" ixz="0.0"/>
+  </inertial>
+  <visual>
+    <origin xyz="-0.0475 -0.0347 -0.067225" rpy="${-pi/2} 0 0"/>
+    <geometry>
+      <mesh filename="package://gonzo_description/meshes/right_tyre.stl" scale="0.001 0.001 0.001"/>
+    </geometry>
+    <material name="tyre_black"/>
+  </visual>
+  <collision>
+    <origin xyz="0.0 0.0 0.013" rpy="0.0 0 0"/>
+    <geometry>
+      <!-- <mesh filename="package://gonzo_description/meshes/right_tyre.stl" scale="0.001 0.001 0.001"/> -->
+      <cylinder radius="0.033" length="0.024"/>
+    </geometry>
+  </collision>
+</link>
+<link name="right_wheel">
+  <inertial>
+    <origin xyz="3.968741960069799e-09 -0.01469275991633777 -1.7434994024900785e-08" rpy="0 0 0"/>
+    <mass value="0.112389434297757225"/>
+    <inertia ixx="3e-04" iyy="5e-04" izz="3e-04" ixy="0.0" iyz="-0.0" ixz="-0.0"/>
+  </inertial>
+  <visual>
+    <origin xyz="-0.0475 -0.0347 -0.067225" rpy="${-pi/2} 0 0"/>
+    <geometry>
+      <mesh filename="package://gonzo_description/meshes/right_wheel.stl" scale="0.001 0.001 0.001"/>
+    </geometry>
+    <material name="yellow"/>
+  </visual>
+  <collision>
+    <origin xyz="-0.0475 -0.0347 -0.067225" rpy="${-pi/2} 0 0"/>
+    <geometry>
+      <mesh filename="package://gonzo_description/meshes/right_wheel.stl" scale="0.001 0.001 0.001"/>
+    </geometry>
+  </collision>
+</link>
+<link name="left_wheel">
+  <inertial>
+    <origin xyz="-7.785304803609172e-09 0.009692764310584537 6.360168114394327e-09" rpy="0 0 0"/>
+    <mass value="0.11238944475891587"/>
+    <inertia ixx="3e-04" iyy="5e-04" izz="3e-04" ixy="-0.0" iyz="0.0" ixz="-0.0"/>
+  </inertial>
+  <visual>
+    <origin xyz="-0.0475 0.0347 -0.067225" rpy="${pi/2} 0 0"/>
+    <geometry>
+      <mesh filename="package://gonzo_description/meshes/left_wheel.stl" scale="0.001 0.001 0.001"/>
+    </geometry>
+    <material name="yellow"/>
+  </visual>
+  <collision>
+    <origin xyz="-0.0475 0.0347 -0.067225" rpy="${pi/2} 0 0"/>
+    <geometry>
+      <mesh filename="package://gonzo_description/meshes/left_wheel.stl" scale="0.001 0.001 0.001"/>
+    </geometry>
+  </collision>
+</link>
+<link name="left_tyre">
+  <inertial>
+    <origin xyz="9.273384204283586e-08 0.017398360785967945 -5.286237849538855e-08" rpy="0 0 0"/>
+    <mass value="0.109430614326368155"/>
+    <inertia ixx="5e-05" iyy="9e-05" izz="5e-05" ixy="-0.0" iyz="0.0" ixz="-0.0"/>
+  </inertial>
+  <visual>
+    <origin xyz="-0.0475 0.0347 -0.067225" rpy="${pi/2} 0 0"/>
+    <geometry>
+      <mesh filename="package://gonzo_description/meshes/left_tyre.stl" scale="0.001 0.001 0.001"/>
+    </geometry>
+    <material name="tyre_black"/>
+  </visual>
+  <collision>
+    <!-- <origin xyz="-0.0475 0.0347 -0.067225" rpy="${pi/2} 0 0"/> -->
+    <origin xyz="0.0 0.0 0.013" rpy="0.0 0 0"/>
+    <geometry>
+      <!-- <mesh filename="package://gonzo_description/meshes/left_tyre.stl" scale="0.001 0.001 0.001"/> -->
+      <cylinder radius="0.033" length="0.024"/>
+    </geometry>
+  </collision>
+</link>
+<link name="right_motor">
+  <inertial>
+    <origin xyz="4.7331206576989304e-07 0.0266233771435831 -1.3780643293159756e-14" rpy="0 0 0"/>
+    <mass value="0.16961662757238829"/>
+    <inertia ixx="2e-05" iyy="5e-06" izz="2e-05" ixy="0.0" iyz="-0.0" ixz="-0.0"/>
+  </inertial>
+  <visual>
+    <origin xyz="-0.0475 0.0601 -0.0347" rpy="0 0 0"/>
+    <geometry>
+      <mesh filename="package://gonzo_description/meshes/right_motor.stl" scale="0.001 0.001 0.001"/>
+    </geometry>
     <material name="silver"/>
   </visual>
   <collision>
-    <origin xyz="0 0 0" rpy="0 0 0"/>
-    <geometry>
-      <mesh filename="package://gonzo_description/meshes/base_link.stl" scale="0.001 0.001 0.001"/>
-    </geometry>
-  </collision>
-</link>
-<link name="right_tyre">
-  <inertial>
-    <origin xyz="-9.273384193181355e-08 -0.017748789854178187 -5.2862379126827896e-08" rpy="0 0 0"/>
-    <mass value="0.009430614326367688"/>
-    <inertia ixx="5e-06" iyy="9e-06" izz="5e-06" ixy="-0.0" iyz="-0.0" ixz="0.0"/>
-  </inertial>
-  <visual>
-    <origin xyz="-0.0475 -0.0347 -0.067225" rpy="${-pi/2} 0 0"/>
-    <geometry>
-      <mesh filename="package://gonzo_description/meshes/right_tyre.stl" scale="0.001 0.001 0.001"/>
+    <origin xyz="-0.0475 0.0601 -0.0347" rpy="0 0 0"/>
+    <geometry>
+      <mesh filename="package://gonzo_description/meshes/right_motor.stl" scale="0.001 0.001 0.001"/>
+    </geometry>
+  </collision>
+</link>
+<link name="left_motor">
+  <inertial>
+    <origin xyz="4.7331206576295415e-07 -0.0266233771435831 1.3787582187063663e-14" rpy="0 0 0"/>
+    <mass value="0.16961662757238826"/>
+    <inertia ixx="2e-05" iyy="5e-06" izz="2e-05" ixy="-0.0" iyz="-0.0" ixz="0.0"/>
+  </inertial>
+  <visual>
+    <origin xyz="-0.0475 -0.0599 -0.0347" rpy="0 0 0"/>
+    <geometry>
+      <mesh filename="package://gonzo_description/meshes/left_motor.stl" scale="0.001 0.001 0.001"/>
     </geometry>
     <material name="silver"/>
   </visual>
   <collision>
-    <origin xyz="-0.0475 -0.0347 -0.067225" rpy="${-pi/2} 0 0"/>
-    <geometry>
-      <mesh filename="package://gonzo_description/meshes/right_tyre.stl" scale="0.001 0.001 0.001"/>
-    </geometry>
-  </collision>
-</link>
-<link name="right_wheel">
-  <inertial>
-    <origin xyz="3.968741960069799e-09 -0.01469275991633777 -1.7434994024900785e-08" rpy="0 0 0"/>
-    <mass value="0.012389434297757225"/>
-    <inertia ixx="3e-06" iyy="5e-06" izz="3e-06" ixy="0.0" iyz="-0.0" ixz="-0.0"/>
-  </inertial>
-  <visual>
-    <origin xyz="-0.0475 -0.0347 -0.067225" rpy="${-pi/2} 0 0"/>
-    <geometry>
-      <mesh filename="package://gonzo_description/meshes/right_wheel.stl" scale="0.001 0.001 0.001"/>
-    </geometry>
-    <material name="silver"/>
-  </visual>
-  <collision>
-    <origin xyz="-0.0475 -0.0347 -0.067225" rpy="${-pi/2} 0 0"/>
-    <geometry>
-      <mesh filename="package://gonzo_description/meshes/right_wheel.stl" scale="0.001 0.001 0.001"/>
-    </geometry>
-  </collision>
-</link>
-<link name="left_wheel">
-  <inertial>
-    <origin xyz="-7.785304803609172e-09 0.009692764310584537 6.360168114394327e-09" rpy="0 0 0"/>
-    <mass value="0.01238944475891587"/>
-    <inertia ixx="3e-06" iyy="5e-06" izz="3e-06" ixy="-0.0" iyz="0.0" ixz="-0.0"/>
-  </inertial>
-  <visual>
-    <origin xyz="-0.0475 0.0347 -0.067225" rpy="${pi/2} 0 0"/>
-    <geometry>
-      <mesh filename="package://gonzo_description/meshes/left_wheel.stl" scale="0.001 0.001 0.001"/>
-    </geometry>
-    <material name="silver"/>
-  </visual>
-  <collision>
-    <origin xyz="-0.0475 0.0347 -0.067225" rpy="${pi/2} 0 0"/>
-    <geometry>
-      <mesh filename="package://gonzo_description/meshes/left_wheel.stl" scale="0.001 0.001 0.001"/>
-    </geometry>
-  </collision>
-</link>
-<link name="left_tyre">
-  <inertial>
-    <origin xyz="9.273384204283586e-08 0.017398360785967945 -5.286237849538855e-08" rpy="0 0 0"/>
-    <mass value="0.009430614326368155"/>
-    <inertia ixx="5e-06" iyy="9e-06" izz="5e-06" ixy="-0.0" iyz="0.0" ixz="-0.0"/>
-  </inertial>
-  <visual>
-    <origin xyz="-0.0475 0.0347 -0.067225" rpy="${pi/2} 0 0"/>
-    <geometry>
-      <mesh filename="package://gonzo_description/meshes/left_tyre.stl" scale="0.001 0.001 0.001"/>
-    </geometry>
-    <material name="silver"/>
-  </visual>
-  <collision>
-    <origin xyz="-0.0475 0.0347 -0.067225" rpy="${pi/2} 0 0"/>
-    <geometry>
-      <mesh filename="package://gonzo_description/meshes/left_tyre.stl" scale="0.001 0.001 0.001"/>
-    </geometry>
-  </collision>
-</link>
-<link name="right_motor">
-  <inertial>
-    <origin xyz="4.7331206576989304e-07 0.0266233771435831 -1.3780643293159756e-14" rpy="0 0 0"/>
-    <mass value="0.06961662757238829"/>
-    <inertia ixx="2e-05" iyy="5e-06" izz="2e-05" ixy="0.0" iyz="-0.0" ixz="-0.0"/>
-  </inertial>
-  <visual>
-    <origin xyz="-0.0475 0.0601 -0.0347" rpy="0 0 0"/>
-    <geometry>
-      <mesh filename="package://gonzo_description/meshes/right_motor.stl" scale="0.001 0.001 0.001"/>
-    </geometry>
-    <material name="silver"/>
-  </visual>
-  <collision>
-    <origin xyz="-0.0475 0.0601 -0.0347" rpy="0 0 0"/>
-    <geometry>
-      <mesh filename="package://gonzo_description/meshes/right_motor.stl" scale="0.001 0.001 0.001"/>
-    </geometry>
-  </collision>
-</link>
-<link name="left_motor">
-  <inertial>
-    <origin xyz="4.7331206576295415e-07 -0.0266233771435831 1.3787582187063663e-14" rpy="0 0 0"/>
-    <mass value="0.06961662757238826"/>
-    <inertia ixx="2e-05" iyy="5e-06" izz="2e-05" ixy="-0.0" iyz="-0.0" ixz="0.0"/>
-  </inertial>
-  <visual>
     <origin xyz="-0.0475 -0.0599 -0.0347" rpy="0 0 0"/>
     <geometry>
       <mesh filename="package://gonzo_description/meshes/left_motor.stl" scale="0.001 0.001 0.001"/>
     </geometry>
-    <material name="silver"/>
-  </visual>
-  <collision>
-    <origin xyz="-0.0475 -0.0599 -0.0347" rpy="0 0 0"/>
-    <geometry>
-      <mesh filename="package://gonzo_description/meshes/left_motor.stl" scale="0.001 0.001 0.001"/>
-    </geometry>
   </collision>
 </link>
@@ -149,6 +152,6 @@
   <inertial>
     <origin xyz="-7.301104165691186e-14 0.01039999999999995 -4.344167282410022e-07" rpy="0 0 0"/>
-    <mass value="0.004208687504738151"/>
-    <inertia ixx="0.0" iyy="0.0" izz="0.0" ixy="0.0" iyz="0.0" ixz="0.0"/>
+    <mass value="0.504208687504738151"/>
+    <inertia ixx="2e-4" iyy="2e-4" izz="2e-4" ixy="0.0" iyz="0.0" ixz="0.0"/>
   </inertial>
   <visual>
@@ -157,10 +160,12 @@
       <mesh filename="package://gonzo_description/meshes/caster_wheel.stl" scale="0.001 0.001 0.001"/>
     </geometry>
-    <material name="silver"/>
-  </visual>
-  <collision>
-    <origin xyz="0.063 0.0105 -0.013814" rpy="0 0 0"/>
-    <geometry>
-      <mesh filename="package://gonzo_description/meshes/caster_wheel.stl" scale="0.001 0.001 0.001"/>
+    <material name="white"/>
+  </visual>
+  <collision>
+    <!-- <origin xyz="0.063 0.0 -0.013814" rpy="0 0 0"/> -->
+    <origin xyz="0.0 0.0 0.0" rpy="0 0 0"/>
+    <geometry>
+      <!-- <mesh filename="package://gonzo_description/meshes/caster_wheel.stl" scale="0.001 0.001 0.001"/> -->
+      <sphere radius="0.015"/>
     </geometry>
   </collision>
@@ -217,5 +222,5 @@
       <mesh filename="package://gonzo_description/meshes/battery_link.stl" scale="0.001 0.001 0.001"/>
     </geometry>
-    <material name="silver"/>
+    <material name="rplidar_black"/>
   </visual>
   <collision>
@@ -237,5 +242,5 @@
       <mesh filename="package://gonzo_description/meshes/raspberry.stl" scale="0.001 0.001 0.001"/>
     </geometry>
-    <material name="silver"/>
+    <material name="white"/>
   </visual>
   <collision>
@@ -249,5 +254,5 @@
   <inertial>
     <origin xyz="0.031039338840954937 0.0003525144946507812 0.08371566276734518" rpy="0 0 0"/>
-    <mass value="0.05976986632824088"/>
+    <mass value="0.35976986632824088"/>
     <inertia ixx="2.4e-05" iyy="5.3e-05" izz="6.2e-05" ixy="-1e-06" iyz="-0.0" ixz="-8e-06"/>
   </inertial>
@@ -257,8 +262,8 @@
       <mesh filename="package://gonzo_description/meshes/laser.dae" scale="0.001 0.001 0.001"/>
     </geometry>
-    <material name="silver"/>
-  </visual>
-  <collision>
-    <origin xyz="0.051 0.0001 -0.0477" rpy="0 0 0"/>
+    <material name="rplidar_black"/>
+  </visual>
+  <collision>
+    <origin xyz="0.005 0.0001 -0.15" rpy="0 0 0"/>
     <geometry>
       <mesh filename="package://gonzo_description/meshes/laser.stl" scale="0.001 0.001 0.001"/>
@@ -267,5 +272,5 @@
 </link>
 <joint name="chassis_joint" type="fixed">
-  <origin xyz="0.0 0.0 0.0" rpy="0.0 0.0 0.0"/>
+  <origin xyz="0.0 0.0 0.05" rpy="0.0 0.0 0.0"/>
   <parent link="base_link"/>
   <child link="chassis_link"/>
@@ -303,15 +308,15 @@
   <child link="left_motor"/>
 </joint>
-<joint name="caster_wheel_joint" type="continuous">
+<joint name="caster_wheel_joint" type="fixed">
   <origin xyz="-0.012 -0.0 -0.021" rpy="0 0 0"/>
   <parent link="caster_holder"/>
   <child link="caster_wheel"/>
-  <axis xyz="0.0 -1.0 -0.0"/>
-</joint>
-<joint name="caster_holder_joint" type="continuous">
+  <!-- <axis xyz="0.0 1.0 0.0"/> -->
+</joint>
+<joint name="caster_holder_joint" type="fixed">
   <origin xyz="0.0 0.0001 -0.060586" rpy="0 0 0"/>
   <parent link="caster_base"/>
   <child link="caster_holder"/>
-  <axis xyz="0.0 -0.0 1.0"/>
+  <!-- <axis xyz="0.0 0.0 1.0"/> -->
 </joint>
 <joint name="caster_base_joint" type="fixed">

File: gonzo_description/urdf/materials.xacro (robot description, xacro)
@@ -4,3 +4,18 @@
   <color rgba="0.700 0.700 0.700 1.000"/>
 </material>
+<material name="white">
+  <color rgba="1.0 1.0 1.0 1.000"/>
+</material>
+<material name="yellow">
+  <color rgba="0.700 0.700 0.00 1.000"/>
+</material>
+<material name="body_black">
+  <color rgba="0.200 0.200 0.200 1.000"/>
+</material>
+<material name="tyre_black">
+  <color rgba="0.100 0.100 0.100 1.000"/>
+</material>
+<material name="rplidar_black">
+  <color rgba="0.250 0.250 0.250 1.000"/>
+</material>
 </robot>

Commit message: Udate gazebo appearence

File: gonzo_description/urdf/gonzo.xacro (robot description, xacro)
@@ -9,6 +9,6 @@
   <inertial>
     <origin xyz="0.004369403453275925 -7.02165131943858e-05 0.06024663017842304" rpy="0 0 0"/>
-    <mass value="5.20273197769577378"/>
-    <inertia ixx="0.0438" iyy="0.0482" izz="0.0751" ixy="0.0" iyz="-0.0" ixz="7e-05"/>
+    <mass value="1.20273197769577378"/>
+    <inertia ixx="0.00438" iyy="0.00482" izz="0.07051" ixy="0.0" iyz="-0.0" ixz="7e-06"/>
   </inertial>
   <visual>
@@ -29,6 +29,6 @@
   <inertial>
     <origin xyz="-9.273384193181355e-08 -0.017748789854178187 -5.2862379126827896e-08" rpy="0 0 0"/>
-    <mass value="1.109430614326367688"/>
-    <inertia ixx="5e-03" iyy="9e-03" izz="5e-03" ixy="-0.0" iyz="-0.0" ixz="0.0"/>
+    <mass value="0.109430614326368155"/>
+    <inertia ixx="5e-05" iyy="9e-05" izz="5e-05" ixy="-0.0" iyz="-0.0" ixz="0.0"/>
   </inertial>
   <visual>
@@ -70,5 +70,5 @@
   <inertial>
     <origin xyz="-7.785304803609172e-09 0.009692764310584537 6.360168114394327e-09" rpy="0 0 0"/>
-    <mass value="0.11238944475891587"/>
+    <mass value="0.112389434297757225"/>
     <inertia ixx="3e-04" iyy="5e-04" izz="3e-04" ixy="-0.0" iyz="0.0" ixz="-0.0"/>
   </inertial>
@@ -112,5 +112,5 @@
   <inertial>
     <origin xyz="4.7331206576989304e-07 0.0266233771435831 -1.3780643293159756e-14" rpy="0 0 0"/>
-    <mass value="0.16961662757238829"/>
+    <mass value="0.1696166275723882"/>
     <inertia ixx="2e-05" iyy="5e-06" izz="2e-05" ixy="0.0" iyz="-0.0" ixz="-0.0"/>
   </inertial>
@@ -132,5 +132,5 @@
   <inertial>
     <origin xyz="4.7331206576295415e-07 -0.0266233771435831 1.3787582187063663e-14" rpy="0 0 0"/>
-    <mass value="0.16961662757238826"/>
+    <mass value="0.1696166275723882"/>
     <inertia ixx="2e-05" iyy="5e-06" izz="2e-05" ixy="-0.0" iyz="-0.0" ixz="0.0"/>
   </inertial>
@@ -152,6 +152,6 @@
   <inertial>
     <origin xyz="-7.301104165691186e-14 0.01039999999999995 -4.344167282410022e-07" rpy="0 0 0"/>
-    <mass value="0.504208687504738151"/>
-    <inertia ixx="2e-4" iyy="2e-4" izz="2e-4" ixy="0.0" iyz="0.0" ixz="0.0"/>
+    <mass value="0.084208687504738151"/>
+    <inertia ixx="2e-6" iyy="2e-6" izz="2e-6" ixy="0.0" iyz="0.0" ixz="0.0"/>
   </inertial>
   <visual>
@@ -194,5 +194,5 @@
   <inertial>
     <origin xyz="-3.863839803663893e-12 9.999999823247428e-05 -0.059707403308328987" rpy="0 0 0"/>
-    <mass value="0.009385654757274695"/>
+    <mass value="0.05385654757274695"/>
     <inertia ixx="1e-06" iyy="1e-06" izz="2e-06" ixy="0.0" iyz="-0.0" ixz="-0.0"/>
   </inertial>
